Commit message: add gazebo files and replaced parts with lower resolution parts

File: src/farmbot_description/urdf/assembly.urdf (robot description, URDF)
Before this commit: robot farmbot, 6 links, 5 joints
Links:
- link cross_slide: mass None -> 1; geometry collision mesh filename=package://farmbot_description/meshes/visual/cross_slide.dae; visual mesh filename=package://farmbot_description/meshes/visual/cross_slide.dae
- link gantry: mass None -> 10; geometry collision mesh filename=package://farmbot_description/meshes/collision/collision_ga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; visual mesh filename=package://farmbot_description/meshes/visual/gantry.dae
- link raised_bed: mass None -> 1; geometry collision box size=1 1 1; visual mesh filename=package://farmbot_description/meshes/visual/raised_bed.dae
- link tracks: mass None -> 10; geometry collision mesh filename=package://farmbot_description/meshes/visual/tracks.dae; visual mesh filename=package://farmbot_description/meshes/visual/tracks.dae
- link z_axis: mass None -> 10; geometry collision mesh filename=package://farmbot_description/meshes/collision/collision_zA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; visual mesh filename=package://farmbot_description/meshes/visual/z_axis.dae
Joints:
- joint joint_cross_slide_z_axis: axis 0 0 1 -> 0 0 -1; limit lower=-0.38 upper=0 effort=1000.0 velocity=0.5 -> lower=-0.38 upper=0.35 effort=1000.0 velocity=0.5

File: src/farmbot_description/urdf/joints/joint_crossSlide_zAxis.urdf (robot description, URDF)
Before this commit: robot fixes_joints, 0 links, 1 joints
Joints:
- joint joint_cross_slide_z_axis: axis 0 0 1 -> 0 0 -1; limit lower=-0.38 upper=0 effort=1000.0 velocity=0.5 -> lower=-0.38 upper=0.35 effort=1000.0 velocity=0.5

File: src/farmbot_description/urdf/joints/joint_crossSlide_zAxis.xacro (robot description, xacro)
@@ -4,6 +4,6 @@
     <parent link="cross_slide"/>
     <child link="z_axis"/>
-    <axis xyz="0 0 1"/>
-    <limit effort="1000.0" lower="-0.38" upper="0" velocity="0.5"/>
+    <axis xyz="0 0 -1"/>
+    <limit effort="1000.0" lower="-0.38" upper="0.35" velocity="0.5"/>
     <origin rpy="0 0 0" xyz="0 0 0"/>
   </joint>

File: src/farmbot_description/urdf/parts/cross_slide.urdf (robot description, URDF)
Before this commit: robot cross_slide, 1 links, 0 joints
Links:
- link cross_slide: mass None -> 1; geometry collision mesh filename=package://farmbot_description/meshes/visual/cross_slide.dae; visual mesh filename=package://farmbot_description/meshes/visual/cross_slide.dae

File: src/farmbot_description/urdf/parts/gantry.urdf (robot description, URDF)
Before this commit: robot gantry, 1 links, 0 joints
Links:
- link gantry: mass None -> 10; geometry collision mesh filename=package://farmbot_description/meshes/collision/collision_ga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; visual mesh filename=package://farmbot_description/meshes/visual/gantry.dae

File: src/farmbot_description/urdf/parts/raised_bed.urdf (robot description, URDF)
Before this commit: robot raised_bed, 1 links, 0 joints
Links:
- link raised_bed: mass None -> 1; geometry collision box size=1 1 1; visual mesh filename=package://farmbot_description/meshes/visual/raised_bed.dae

File: src/farmbot_description/urdf/parts/tracks.urdf (robot description, URDF)
Before this commit: robot tracks, 1 links, 0 joints
Links:
- link tracks: mass None -> 10; geometry collision mesh filename=package://farmbot_description/meshes/visual/tracks.dae; visual mesh filename=package://farmbot_description/meshes/visual/tracks.dae

File: src/farmbot_description/urdf/parts/z_axis.urdf (robot description, URDF)
Before this commit: robot z_axis, 1 links, 0 joints
Links:
- link z_axis: mass None -> 10; geometry collision mesh filename=package://farmbot_description/meshes/collision/collision_zA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; visual mesh filename=package://farmbot_description/meshes/visual/z_axis.dae

File: src/farmbot_description/urdf/tests/assembly_gantry_crossSlide.urdf (robot description, URDF)
Before this commit: robot farmbot, 3 links, 2 joints
Links:
- link cross_slide: mass None -> 1
